File: pcb/kicad/projects/BMEK_Hotswap/BMEK_Hotswap.kicad_sch (KiCad schematic)
At the start: 188 parts, among them J1 Conn_01x04, J2 AVR-ISP-6, SW1 TS-1187A-B-A-B, U1 ATmega32U4-AU, U2 USBLC6-2SC6, Y1 Crystal_GND24_Small

Commit message: Crosshatch / normal version
Parts:
- V1: footprint BMEK:PCBProfile_NO_Switches_copy -> BMEK:PCBProfile_NO_Switches
Changed lines of the file:
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@@
   (junction (at 379.857 164.719) (diameter 1.016) (color 0 0 0 0))
   (junction (at 384.937 152.019) (diameter 1.016) (color 0 0 0 0))
-  (no_connect (at 34.798 52.324))
   (no_connect (at 34.798 37.084))
+  (no_connect (at 377.444 29.972))
   (no_connect (at 167.894 31.369))
+  (no_connect (at 34.798 52.324))
   (no_connect (at 162.814 51.689))
-  (no_connect (at 377.444 29.972))
   (wire (pts (xy 23.241 165.989) (xy 39.751 165.989))
     (stroke (width 0) (type solid) (color 0 0 0 0))
@@
     )
     (property "Value" "PCBProfile" (id 1) (at 125.9586 23.1394 0))
-    (property "Footprint" "BMEK:PCBProfile_NO_Switches_copy" (id 2) (at 117.3226 27.9654 0)
+    (property "Footprint" "BMEK:PCBProfile_NO_Switches" (id 2) (at 117.3226 27.9654 0)
       (effects (font (size 1.27 1.27)) hide)
     )
